File: stlink-power-supply/stlink-power-supply.kicad_pcb (KiCad board)
At the start: 2 copper layers, 50.8 x 36.8 mm, 12 parts, among them J1 USB_B, J2 STLinkV3-MINI, J3 STLinkV3-MINI, U1 OKL-T6-W12

Commit message: add another interface
Parts:
- added J4: DEBUG, Connector_IDC:IDC-Header_2x05_P2.54mm_Vertical, F.Cu at (135.9, 89.5)
- added J5: out, Connector_JST:JST_PH_B2B-PH-K_1x02_P2.00mm_Vertical, F.Cu at (126.4, 116.7)
- added J6: out, Connector_JST:JST_PH_B2B-PH-K_1x02_P2.00mm_Vertical, F.Cu at (126.4, 125.7)
- added J7: out, Connector_JST:JST_XH_B2B-XH-AM_1x02_P2.50mm_Vertical, F.Cu at (125.7, 106.0)
- added J8: out, Connector_JST:JST_XH_B2B-XH-AM_1x02_P2.50mm_Vertical, F.Cu at (125.7, 95.9)
- moved J2 28.4 mm to (170.2, 88.9)
- moved J3 13.7 mm to (177.8, 95.2), turned to 0 degrees
Connections:
- J2 pad 8: GND -> /SWO
- J3 pad 8: GND -> /SWO
Routing:
- net +3V3: track 33.6 -> 119.8 mm, vias 0 -> 1
- net /SWO: track 0.00 -> 47.1 mm, vias 0 -> 1
- net GND: track 164.4 -> 202.1 mm, vias 0 -> 1
- net /SWCLK: track 44.5 -> 72.8 mm, vias 0 -> 3
- net /SWDIO: track 24.8 -> 44.3 mm, vias 2 -> 5
- net /RST: track 45.6 -> 57.5 mm, vias 0 -> 3
- net /TX: track 42.6 -> 47.6 mm, vias 1 -> 3
- net /RX: track 39.7 -> 43.8 mm, vias 0 -> 2
- removed copper zone on B.Cu, net GND
Other:
- board size 50.8 x 36.8 mm -> 59.7 x 47 mm
- rule trace_min: 0.2 -> 0
